File: Arduino/PCB/SigFoxBatteryMonitor.sch (EAGLE design)
At the start: 55 parts, among them IC1 BD6211F, IC2 BD6211F, IC3 7805TV, Q1 MOSFET-NCHANNELFDS6630A, Q2 MOSFET-NCHANNELFDS6630A, Q3 MOSFET-NCHANNELFDS6630A, U1 INA219AIDCNRSOIC, X2 PN87520-S

Commit message: Version 1.0 PCB.
Parts:
- added D3, D4: MBRA140, SparkFun-DiscreteSemi:DIODE-SCHOTTKY-MBRA140
- added JP12, JP13, JP14: (no value), SparkFun-Connectors:M02PTH
- added JP15, JP16, JP17, JP18, JP19, JP20, JP21, JP22, JP23, JP25, JP26, JP27, JP28, JP29, JP30, JP31: (no value), SparkFun-Connectors:M05NO_SILK
- added JP32, JP33: (no value), SparkFun-Connectors:M05PTH
- added R10, R9: 100k, SparkFun-Resistors:RESISTOR0805
- added R11, R12, R13, R14, R15, R16: (no value), SparkFun-Resistors:RESISTOR0805
- added TP4: 5v, testpad:TPTP15R
- BATTERY, CHARGE, OUTPUT: FARNELL (none) -> 2493689
- C1, C2: FARNELL (none) -> 1457413
- C9: value 1.0uF -> 0.1uF
- IC1, IC2: FARNELL (none) -> 1716256
- JP7: device SparkFun-Connectors:M03POLAR -> SparkFun-Connectors:M04POLAR
- JP8: device SparkFun-Connectors:M03POLAR -> SparkFun-Connectors:M01PTH
- Q1, Q2, Q3: value MOSFET-NCHANNELFDS6630A -> IRF7413Z; FARNELL (none) -> 2468020
- R1: value (none) -> 1k5
- R3, R5, R7: value (none) -> 10R
- R4, R6, R8: value (none) -> 10k
- U$1, U$2: FARNELL (none) -> 2432863
- U2: value (none) -> 1117st33; FARNELL (none) -> 1652366
Connections:
- new net A5: JP10.8, R13.2, R14.1, U$3.A5
- new net A6: JP10.7, R15.2, R16.1, U$3.A6
- new net N$14: D3.C, JP12.2
- new net N$16: JP8.1, R9.2
- new net N$18: D2.A, JP14.1
- new net N$19: C3.1, C4.1, D4.A, TP4.TP, U2.OUT, U2.OUT@1
- net +3V3: now also D4.C, JP12.1; no longer C3.1, C4.1, JP7.3, JP8.3, U2.OUT, U2.OUT@1
- net 5V: now also JP13.2, JP7.4
- net ANALOG_0: now also R10.2, R9.1
- net ANALOG_5: now also R13.1; no longer JP10.8, U$3.A5
- net ANALOG_6: now also JP7.3, R15.1; no longer JP10.7, JP8.2, U$3.A6
- net ARDUINO_5V: now also JP13.1
- net GND: now also JP33.1, JP33.2, JP33.3, JP33.4, JP33.5, R10.1, R14.2, R16.2; no longer JP8.1
- net SCL: now also R12.1
- net SDA: now also R11.1
- net VCC: now also D3.A, JP32.1, JP32.2, JP32.3, JP32.4, JP32.5, R11.2, R12.2, U$3.3V3; no longer U$3.VCC
- net V_BATT: now also JP14.2; no longer D2.A
Other:
- note added: "5V Safe inputs"
- note added: "Analog 1 or 2 can be interrputs"
- note added: "Battery +ve for batt level sense"
- note added: "Connect for onboard regulators. Default to connected."
- note added: "Connect if not using onboard 3v3 regulator"
- note added: "Connect if not using onboard 5V regulator"
- moved on the sheet: C4, C7, TP1, TP2

Commit message: Fixed type on silkscreen and improved layout of schematic.
Other:
- note added: "Prototype area"
- moved on the sheet: C3, C4, C5, C6, C7, D2, D3, D4, IC3, JP10, JP11, JP12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
